Commit message: Add lidar simulation.

File: sfframework_simulation/descriptions/rbkairos_with_lidar.urdf.xacro (robot description, xacro)
@@ -66,21 +66,52 @@
       rpy="0 0 0" />
   </xacro:sensor_intel_realsense_d435>
-  <link name="test_cube_link">
-    <visual>
-      <geometry> <box size="1 1 1"/> </geometry>
-      <material name="debug_blue"> <color rgba="0 0 1 1"/> </material>
-    </visual>
-    <collision>
-      <geometry> <box size="0.1 0.1 0.1"/> </geometry>
-    </collision>
+<link name="$(arg prefix)top_lidar_link">
     <inertial>
       <mass value="0.1"/>
       <inertia ixx="0.0001" ixy="0" ixz="0" iyy="0.0001" iyz="0" izz="0.0001"/>
     </inertial>
+    <visual>
+      <geometry> <cylinder length="0.14" radius="0.04"/> </geometry>
+      <material name="black"> <color rgba="0 0 0 1"/> </material>
+    </visual>
+    <collision>
+      <geometry> <cylinder length="0.14" radius="0.04"/> </geometry>
+    </collision>
   </link>
-  <joint name="robot_to_cube_joint" type="fixed">
+  <joint name="$(arg prefix)top_lidar_joint" type="fixed">
     <parent link="$(arg prefix)base_link" />
-    <child link="test_cube_link" />
-    <origin xyz="0 0 1.0" rpy="0 0 0" />
+    <child link="$(arg prefix)top_lidar_link" />
+    <origin xyz="0 0 1" rpy="0 0 0" />
   </joint>
+  <gazebo reference="$(arg prefix)top_lidar_link">
+    <sensor name="top_lidar" type="gpu_lidar">
+      <pose>0 0 0 0 0 0</pose>
+      <topic>$(arg prefix)top_lidar/scan/points</topic>
+      <gz_frame_id>$(arg prefix)top_lidar_link</gz_frame_id>
+      <update_rate>10</update_rate>
+      <visualize>true</visualize>
+      <lidar>
+        <scan>
+          <horizontal>
+            <samples>1024</samples>
+            <resolution>1</resolution>
+            <min_angle>-3.14159</min_angle>
+            <max_angle>3.14159</max_angle>
+          </horizontal>
+          <vertical>
+            <samples>32</samples> <resolution>1</resolution>
+            <min_angle>-0.535</min_angle> <max_angle>0.186</max_angle>  </vertical>
+        </scan>
+        <range>
+          <min>0.3</min>
+          <max>80.0</max>
+        </range>
+        <noise>
+          <type>gaussian</type>
+          <mean>0.0</mean>
+          <stddev>0.02</stddev> <!-- from the specs: "Range accuracy: <20mm"-->
+        </noise>
+      </lidar>
+    </sensor>
+  </gazebo>
 </robot>
